Commit message: end m3 task

File: urdf/planar2dof.urdf (robot description, URDF)
Before this commit: robot planar2dof, 5 links, 4 joints
Links:
- link planar2dof/link_2: mass 2.4 -> 2.5
- link planar2dof/link_striker_ee: mass 0.1 -> 0.0

Commit message: feedback linearization done

File: urdf/planar2dof.urdf (robot description, URDF)
Before this commit: robot planar2dof, 5 links, 4 joints
Links:
- link planar2dof/link_2: mass 2.5 -> 2.9

Commit message: end finaly first starting second, stop on choose model

File: urdf/planar2dof.urdf (robot description, URDF)
Before this commit: robot planar2dof, 5 links, 4 joints
Links:
- link planar2dof/link_2: mass 2.9 -> 2.4
- link planar2dof/link_striker_ee: mass 0.0 -> 0.5
